Commit message: Imported upstream version '0.0.3' of 'upstream'

File: clearpath_platform_description/urdf/a200/a200.urdf.xacro (robot description, xacro)
@@ -15,5 +15,5 @@
     <!-- Wheel Mounting Positions -->
     <xacro:property name="wheelbase" value="0.5120" />
-    <xacro:property name="track" value="0.5708" />
+    <xacro:property name="track" value="0.555" />
     <xacro:property name="wheel_vertical_offset" value="0.03282" />
     <!-- Wheel Properties -->
@@ -88,4 +88,32 @@
       <origin xyz="${-wheelbase/2} ${-track/2} ${wheel_vertical_offset}" rpy="0 0 0" />
     </xacro:a200_wheel>
+    <gazebo>
+      <plugin filename="libignition-gazebo-wheel-slip-system.so" name="ignition::gazebo::systems::WheelSlip">
+        <wheel link_name="front_left_wheel">
+          <slip_compliance_lateral>1.0</slip_compliance_lateral>
+          <slip_compliance_longitudinal>1.0</slip_compliance_longitudinal>
+          <wheel_normal_force>113</wheel_normal_force>
+          <wheel_radius>${wheel_radius}</wheel_radius>
+        </wheel>
+        <wheel link_name="front_right_wheel">
+          <slip_compliance_lateral>1.0</slip_compliance_lateral>
+          <slip_compliance_longitudinal>1.0</slip_compliance_longitudinal>
+          <wheel_normal_force>113</wheel_normal_force>
+          <wheel_radius>${wheel_radius}</wheel_radius>
+        </wheel>
+        <wheel link_name="rear_left_wheel">
+          <slip_compliance_lateral>1.0</slip_compliance_lateral>
+          <slip_compliance_longitudinal>1.0</slip_compliance_longitudinal>
+          <wheel_normal_force>113</wheel_normal_force>
+          <wheel_radius>${wheel_radius}</wheel_radius>
+        </wheel>
+        <wheel link_name="rear_right_wheel">
+          <slip_compliance_lateral>1.0</slip_compliance_lateral>
+          <slip_compliance_longitudinal>1.0</slip_compliance_longitudinal>
+          <wheel_normal_force>113</wheel_normal_force>
+          <wheel_radius>${wheel_radius}</wheel_radius>
+        </wheel>
+      </plugin>
+    </gazebo>
     <!-- Front bumper mount -->
     <link name="front_bumper_mount"/>

File: clearpath_platform_description/urdf/a200/wheel.urdf.xacro (robot description, xacro)
@@ -21,11 +21,11 @@
       </collision>
     </link>
-    <gazebo reference="${wheel_prefix}_wheel">
+    <!-- <gazebo reference="${wheel_prefix}_wheel">
       <mu1 value="1.0"/>
-      <mu2 value="0.1"/>
-      <kp value="10000000000.0" />
-      <kd value="1000.0" />
+      <mu2 value="0.5"/>
+      <kp value="100000000000000000000.0" />
+      <kd value="1.0" />
       <fdir1 value="1 0 0"/>
-    </gazebo>
+    </gazebo> -->
     <joint name="${wheel_prefix}_wheel_joint" type="continuous">
       <parent link="base_link"/>

File: clearpath_platform_description/urdf/j100/j100.urdf.xacro (robot description, xacro)
@@ -32,4 +32,32 @@
       <origin xyz="${-wheelbase/2} ${-track/2} ${wheel_vertical_offset}" rpy="0 0 0" />
     </xacro:j100_wheel>
+    <gazebo>
+      <plugin filename="libignition-gazebo-wheel-slip-system.so" name="ignition::gazebo::systems::WheelSlip">
+        <wheel link_name="front_left_wheel_link">
+          <slip_compliance_lateral>1.0</slip_compliance_lateral>
+          <slip_compliance_longitudinal>1.0</slip_compliance_longitudinal>
+          <wheel_normal_force>40</wheel_normal_force>
+          <wheel_radius>${wheel_radius}</wheel_radius>
+        </wheel>
+        <wheel link_name="front_right_wheel_link">
+          <slip_compliance_lateral>1.0</slip_compliance_lateral>
+          <slip_compliance_longitudinal>1.0</slip_compliance_longitudinal>
+          <wheel_normal_force>40</wheel_normal_force>
+          <wheel_radius>${wheel_radius}</wheel_radius>
+        </wheel>
+        <wheel link_name="rear_left_wheel_link">
+          <slip_compliance_lateral>1.0</slip_compliance_lateral>
+          <slip_compliance_longitudinal>1.0</slip_compliance_longitudinal>
+          <wheel_normal_force>40</wheel_normal_force>
+          <wheel_radius>${wheel_radius}</wheel_radius>
+        </wheel>
+        <wheel link_name="rear_right_wheel_link">
+          <slip_compliance_lateral>1.0</slip_compliance_lateral>
+          <slip_compliance_longitudinal>1.0</slip_compliance_longitudinal>
+          <wheel_normal_force>40</wheel_normal_force>
+          <wheel_radius>${wheel_radius}</wheel_radius>
+        </wheel>
+      </plugin>
+    </gazebo>
     <link name="base_link"></link>
     <joint name="base_link_joint" type="fixed">

File: clearpath_platform_description/urdf/j100/wheel.urdf.xacro (robot description, xacro)
@@ -19,8 +19,5 @@
         <origin xyz="0 0 0" rpy="0 0 0"/>
         <mass value="0.477"/>
-        <inertia
-          ixx="0.0013" ixy="0" ixz="0"
-          iyy="0.0024" iyz="0"
-          izz="0.0013"/>
+        <inertia ixx="0.0013" ixy="0" ixz="0" iyy="0.0024" iyz="0" izz="0.0013"/>
       </inertial>
     </link>
@@ -28,8 +25,6 @@
       <material>Gazebo/DarkGrey</material>
       <selfCollide>false</selfCollide>
-      <mu1 value="1.0"/>
-      <mu2 value="0.4"/>
-      <kp value="10000000000.0" />
-      <kd value="1000.0" />
+      <mu1 value="0.5"/>
+      <mu2 value="0.5"/>
       <fdir1 value="1 0 0"/>
     </gazebo>
