Commit message: Imported upstream version '0.0.7' of 'upstream'

File: clearpath_platform_description/urdf/a200/attachments/bumper.urdf.xacro (robot description, xacro)
@@ -10,5 +10,5 @@
             <visual>
                 <geometry>
-                    <mesh filename="package://clearpath_platform_description/meshes/a200/decorations/bumper.dae" />
+                    <mesh filename="package://clearpath_platform_description/meshes/a200/attachments/bumper.dae" />
                 </geometry>
             </visual>

File: clearpath_platform_description/urdf/a200/attachments/front_bumper.urdf.xacro (robot description, xacro)
@@ -6,5 +6,5 @@
             <visual>
                 <geometry>
-                <mesh filename="package://clearpath_platform_description/meshes/a200/decorations/bumper.dae" />
+                <mesh filename="package://clearpath_platform_description/meshes/a200/attachments/bumper.dae" />
                 </geometry>
             </visual>
@@ -20,5 +20,5 @@
                 <visual>
                     <geometry>
-                        <mesh filename="package://clearpath_platform_description/meshes/a200/decorations/bumper_extension.dae" />
+                        <mesh filename="package://clearpath_platform_description/meshes/a200/attachments/bumper_extension.dae" />
                     </geometry>
                 </visual>

File: clearpath_platform_description/urdf/a200/attachments/rear_bumper.urdf.xacro (robot description, xacro)
@@ -6,5 +6,5 @@
         <visual>
             <geometry>
-            <mesh filename="package://clearpath_platform_description/meshes/a200/decorations/bumper.dae" />
+            <mesh filename="package://clearpath_platform_description/meshes/a200/attachments/bumper.dae" />
             </geometry>
         </visual>
@@ -20,5 +20,5 @@
                 <visual>
                     <geometry>
-                        <mesh filename="package://clearpath_platform_description/meshes/a200/decorations/bumper_extension.dae" />
+                        <mesh filename="package://clearpath_platform_description/meshes/a200/attachments/bumper_extension.dae" />
                     </geometry>
                 </visual>

File: clearpath_platform_description/urdf/a200/attachments/structure.urdf.xacro (robot description, xacro)
@@ -8,5 +8,5 @@
           <origin xyz="0 0 0.51" rpy="0 0 0"/>
           <geometry>
-            <mesh filename="package://clearpath_platform_description/meshes/a200/decorations/510_mm_sensor_arch.dae" />
+            <mesh filename="package://clearpath_platform_description/meshes/a200/attachments/510_mm_sensor_arch.dae" />
           </geometry>
         </visual>
@@ -14,5 +14,5 @@
           <origin xyz="0 0 0.51" rpy="0 0 0"/>
           <geometry>
-            <mesh filename="package://clearpath_platform_description/meshes/a200/decorations/510_mm_sensor_arch.dae" />
+            <mesh filename="package://clearpath_platform_description/meshes/a200/attachments/510_mm_sensor_arch.dae" />
           </geometry>
         </collision>
@@ -37,5 +37,5 @@
           <origin xyz="0 0 0.3" rpy="0 0 0"/>
           <geometry>
-            <mesh filename="package://clearpath_platform_description/meshes/a200/decorations/300_mm_sensor_arch.dae" />
+            <mesh filename="package://clearpath_platform_description/meshes/a200/attachments/300_mm_sensor_arch.dae" />
           </geometry>
         </visual>
@@ -43,5 +43,5 @@
           <origin xyz="0 0 0.3" rpy="0 0 0"/>
           <geometry>
-            <mesh filename="package://clearpath_platform_description/meshes/a200/decorations/300_mm_sensor_arch.dae" />
+            <mesh filename="package://clearpath_platform_description/meshes/a200/attachments/300_mm_sensor_arch.dae" />
           </geometry>
         </collision>

File: clearpath_platform_description/urdf/a200/attachments/top_plate.urdf.xacro (robot description, xacro)
@@ -9,5 +9,5 @@
             <origin xyz="0 0 0" rpy="0 0 0" />
             <geometry>
-              <mesh filename="package://clearpath_platform_description/meshes/a200/decorations/large_top_plate.dae" />
+              <mesh filename="package://clearpath_platform_description/meshes/a200/attachments/large_top_plate.dae" />
             </geometry>
           </visual>
@@ -15,5 +15,5 @@
             <origin xyz="0 0 0" rpy="0 0 0"/>
             <geometry>
-              <mesh filename="package://clearpath_platform_description/meshes/a200/decorations/large_top_plate_collision.stl" />
+              <mesh filename="package://clearpath_platform_description/meshes/a200/attachments/large_top_plate_collision.stl" />
             </geometry>
           </collision>
@@ -45,5 +45,5 @@
             <origin xyz="0 0 0" rpy="0 0 0" />
             <geometry>
-              <mesh filename="package://clearpath_platform_description/meshes/a200/decorations/top_plate.dae" />
+              <mesh filename="package://clearpath_platform_description/meshes/a200/attachments/top_plate.dae" />
             </geometry>
           </visual>
@@ -51,5 +51,5 @@
             <origin xyz="0 0 0" rpy="0 0 0"/>
             <geometry>
-              <mesh filename="package://clearpath_platform_description/meshes/a200/decorations/top_plate.stl" />
+              <mesh filename="package://clearpath_platform_description/meshes/a200/attachments/top_plate.stl" />
             </geometry>
           </collision>
@@ -77,5 +77,5 @@
           <visual>
             <geometry>
-              <mesh filename="package://clearpath_platform_description/meshes/a200/decorations/user_rail.dae" />
+              <mesh filename="package://clearpath_platform_description/meshes/a200/attachments/user_rail.dae" />
             </geometry>
           </visual>
@@ -95,5 +95,5 @@
             <material name="dark_grey" />
             <geometry>
-              <mesh filename="package://clearpath_platform_description/meshes/a200/decorations/pacs_top_plate.stl" />
+              <mesh filename="package://clearpath_platform_description/meshes/a200/attachments/pacs_top_plate.stl" />
             </geometry>
           </visual>

File: clearpath_platform_description/urdf/j100/attachments/bumper.urdf.xacro (robot description, xacro)
@@ -10,5 +10,5 @@
       <visual>
         <geometry>
-          <mesh filename="package://clearpath_platform_description/meshes/j100/decorations/j100_fender.stl" />
+          <mesh filename="package://clearpath_platform_description/meshes/j100/attachments/j100_fender.stl" />
         </geometry>
         <material name="yellow" />

File: clearpath_platform_description/urdf/j100/attachments/top_plate.urdf.xacro (robot description, xacro)
@@ -7,5 +7,5 @@
             <origin xyz="0 0 0" rpy="0 0 0"/>
             <geometry>
-              <mesh filename="package://clearpath_platform_description/meshes/j100/decorations/ark_enclosure.stl"/>
+              <mesh filename="package://clearpath_platform_description/meshes/j100/attachments/ark_enclosure.stl"/>
             </geometry>
             <material name="dark_grey" />

File: clearpath_platform_description/urdf/links/frame.urdf.xacro (robot description, xacro)
@@ -1,5 +1,5 @@
 <?xml version="1.0"?>
 <robot xmlns:xacro="http://ros.org/wiki/xacro">
-  <xacro:macro name="link" params="name parent_link *origin">
+  <xacro:macro name="frame" params="name parent_link *origin">
     <link name="${name}_link"/>
     <joint name="${name}_joint" type="fixed">
