Commit message: Imported upstream version '0.2.1' of 'upstream'

File: clearpath_platform_description/urdf/a200/attachments/top_plate.urdf.xacro (robot description, xacro)
@@ -98,5 +98,5 @@
         <link name="${name}_link">
           <visual>
-            <origin xyz="0.0483 0 0"/>
+            <origin xyz="0 0 0"/>
             <material name="clearpath_dark_grey" />
             <geometry>
@@ -106,5 +106,5 @@
           <collision>
             <material name="clearpath_dark_grey" />
-            <origin xyz="0.0483 0 0.003175" rpy="0 0 0"/>
+            <origin xyz="0 0 0.003175" rpy="0 0 0"/>
             <geometry>
               <box size="0.67 0.59 0.00635"/>

Commit message: Imported upstream version '0.2.7' of 'upstream'

File: clearpath_platform_description/urdf/a200/attachments/top_plate.urdf.xacro (robot description, xacro)
@@ -25,4 +25,11 @@
           <xacro:insert_block name="origin"/>
         </joint>
+        <!-- Top plate default link -->
+        <link name="${name}_default_mount"/>
+        <joint name="${name}_default_joint" type="fixed">
+          <parent link="${name}_link" />
+          <child link="${name}_default_mount"/>
+          <origin xyz="0.0812 0 0.00672" rpy="0 0 0"/>
+        </joint>
         <!-- Top plate front link -->
         <link name="${name}_front_mount"/>
@@ -30,5 +37,5 @@
           <parent link="${name}_link" />
           <child link="${name}_front_mount"/>
-          <origin xyz="0.4125 0 0.00672" rpy="0 0 0"/>
+          <origin xyz="0.4937 0 0.00672" rpy="0 0 0"/>
         </joint>
         <!-- Top plate rear link-->
@@ -37,5 +44,5 @@
           <parent link="${name}_link" />
           <child link="${name}_rear_mount"/>
-          <origin xyz="-0.4125 0 0.00672" rpy="0 0 0"/>
+          <origin xyz="-0.3313 0 0.00672" rpy="0 0 0"/>
         </joint>
       </xacro:if>
@@ -78,4 +85,11 @@
           <origin xyz="0 0 0.021" rpy="0 0 0"/>
         </joint>
+        <!-- Top plate default link -->
+        <link name="${name}_default_mount"/>
+        <joint name="${name}_default_joint" type="fixed">
+          <parent link="${name}_link" />
+          <child link="${name}_default_mount"/>
+          <origin xyz="0.07987 0 0.00639" rpy="0 0 0"/>
+        </joint>
         <!-- Top plate front link -->
         <link name="${name}_front_mount"/>
@@ -83,5 +97,5 @@
           <parent link="${name}_link" />
           <child link="${name}_front_mount"/>
-          <origin xyz="0.36367 0 0.00639" rpy="0 0 0"/>
+          <origin xyz="0.44487 0 0.00639" rpy="0 0 0"/>
         </joint>
         <!-- Top plate rear link-->
@@ -90,5 +104,5 @@
           <parent link="${name}_link" />
           <child link="${name}_rear_mount"/>
-          <origin xyz="-0.36633 0 0.00639" rpy="0 0 0"/>
+          <origin xyz="-0.28513 0 0.00639" rpy="0 0 0"/>
         </joint>
       </xacro:if>
@@ -96,4 +110,5 @@
       <xacro:if value="${model == 'pacs'}">
         <!-- Spawn top plate -->
+        <link name="${name}_adjust_link"/>
         <link name="${name}_link">
           <visual>
@@ -113,8 +128,13 @@
         </link>
         <!-- Attach PACS top plate -->
+        <joint name="${name}_adjust_joint" type="fixed">
+          <child link="${name}_adjust_link"/>
+          <parent link="${parent_link}"/>
+          <xacro:insert_block name="origin"/>
+        </joint>
         <joint name="${name}_joint" type="fixed">
           <child link="${name}_link"/>
-          <parent link="${parent_link}"/>
-          <xacro:insert_block name="origin"/>
+          <parent link="${name}_adjust_link"/>
+          <origin xyz="0.04825 0.0 0.0" rpy="0.0 0.0 0.0"/>
         </joint>
         <!-- Generate PACS mounts -->

File: clearpath_platform_description/urdf/w200/attachments/arm_plate.urdf.xacro (robot description, xacro)
@@ -1,5 +1,5 @@
 <?xml version="1.0"?>
 <robot xmlns:xacro="http://ros.org/wiki/xacro">
-  <xacro:macro name="arm_mount" params="name:=arm_mount model:=default parent_link:=default_mount *origin">
+  <xacro:macro name="arm_plate" params="name:=arm_plate model:=default parent_link:=default_mount *origin">
     <link name="${name}_link">
       <visual>
@@ -27,4 +27,10 @@
       <child link="${name}_link" />
     </joint>
+    <link name="${name}_mount"/>
+    <joint name="${name}_mount_joint" type="fixed">
+      <origin xyz="0 0 0.02" rpy="0 0 0"/>
+      <parent link="${name}_link"/>
+      <child link="${name}_mount"/>
+    </joint>
   </xacro:macro>
 </robot>

File: clearpath_platform_description/urdf/w200/attachments/bulkhead.urdf.xacro (robot description, xacro)
@@ -2,8 +2,8 @@
 <robot xmlns:xacro="http://www.ros.org/wiki/xacro">
   <xacro:macro name="bulkhead" params="name:=bulkhead model:=default parent_link:=default_mount *origin">
-    <xacro:include filename="$(find clearpath_platform_description)/urdf/w200/attachments/arm_mount.urdf.xacro"/>
+    <xacro:include filename="$(find clearpath_platform_description)/urdf/w200/attachments/arm_plate.urdf.xacro"/>
     <link name="${name}_link">
       <visual>
-        <origin xyz="0 0 0" rpy="0 0 0"/>
+        <origin xyz="0.00705 0 0.24184" rpy="0 0 0"/>
         <geometry>
           <mesh filename="package://clearpath_platform_description/meshes/w200/bulkhead.stl" />
@@ -12,5 +12,5 @@
       </visual>
       <collision>
-        <origin xyz="0 0 0" rpy="0 0 0"/>
+        <origin xyz="0.00705 0 0.24184" rpy="0 0 0"/>
         <geometry>
           <mesh filename="package://clearpath_platform_description/meshes/w200/bulkhead-collision.stl" />
@@ -28,14 +28,14 @@
       <child link="${name}_link" />
     </joint>
-    <link name="${name}_front_mount_link"/>
-    <joint name="${name}_front_mount_link_joint" type="fixed">
-      <origin xyz="0.33987 0 0.0" rpy="0 0 0" />
+    <link name="${name}_mount"/>
+    <joint name="${name}_mount_joint" type="fixed">
+      <origin xyz="0.34692 0 0.24184" rpy="0 0 0" />
       <parent link="${name}_link"/>
-      <child link="${name}_front_mount_link" />
+      <child link="${name}_mount" />
     </joint>
-    <xacro:if value="${model == 'arm_mount'}">
-      <xacro:arm_mount parent_link="${name}_front_mount_link">
+    <xacro:if value="${model == 'arm_plate'}">
+      <xacro:arm_plate parent_link="${name}_mount">
         <origin xyz="0.0 0.0 0.0" rpy="0.0 0.0 0.0"/>
-      </xacro:arm_mount>
+      </xacro:arm_plate>
     </xacro:if>
   </xacro:macro>

File: clearpath_platform_description/urdf/w200/attachments/generator.urdf.xacro (robot description, xacro)
@@ -4,5 +4,5 @@
     <link name="${name}_link">
       <visual>
-        <origin xyz="0 0 0" rpy="0 0 0"/>
+        <origin xyz="-0.42506 0.0 0.0017" rpy="0 0 0"/>
         <geometry>
           <mesh filename="package://clearpath_platform_description/meshes/w200/generator.stl" />
@@ -11,5 +11,5 @@
       </visual>
       <collision>
-        <origin xyz="0 0 0" rpy="0 0 0"/>
+        <origin xyz="-0.42506 0.0 0.0017" rpy="0 0 0"/>
         <geometry>
           <mesh filename="package://clearpath_platform_description/meshes/w200/generator.stl" />
