Commit message: Imported upstream version '0.0.8' of 'upstream'

File: clearpath_platform_description/urdf/j100/j100.urdf.xacro (robot description, xacro)
@@ -92,5 +92,5 @@
        always points to the "active" IMU. When an upgrade IMU is connected, the
        internal_imu_link should remain, but imu_link should point to the upgrade one. -->
-    <link name="imu_link">
+    <link name="imu_0_link">
       <inertial>
         <mass value="0.001"/>
@@ -101,8 +101,8 @@
     <joint name="imu_joint" type="fixed">
       <parent link="chassis_link" />
-      <child link="imu_link" />
-    </joint>
-    <gazebo reference="imu_link">
-      <sensor type="imu" name="imu_link">
+      <child link="imu_0_link" />
+    </joint>
+    <gazebo reference="imu_0_link">
+      <sensor type="imu" name="imu_0_link">
         <always_on>true</always_on>
         <update_rate>50</update_rate>
@@ -111,5 +111,5 @@
     </gazebo>
     <!-- TODO: Same note as applies to imu_link -->
-    <link name="navsat_link">
+    <link name="gps_0_link">
       <visual>
         <geometry>
@@ -122,9 +122,9 @@
     <joint name="navsat_joint" type="fixed">
       <parent link="chassis_link" />
-      <child link="navsat_link" />
+      <child link="gps_0_link" />
       <origin xyz="-0.180 0.126 0.1815" />
     </joint>
-    <gazebo reference="navsat_link">
-      <sensor name="navsat_link" type="navsat">
+    <gazebo reference="gps_0_link">
+      <sensor name="gps_0_link" type="navsat">
         <always_on>1</always_on>
         <update_rate>10</update_rate>
