Commit message: Imported upstream version '0.0.9' of 'upstream'

File: clearpath_sensors_description/urdf/garmin_18x.urdf.xacro (robot description, xacro)
@@ -1,19 +1,16 @@
 <?xml version="1.0"?>
 <robot xmlns:xacro="http://www.ros.org/wiki/xacro">
-  <xacro:macro name="novatel_smart7" params="name parent_link *origin">
+  <xacro:macro name="garmin_18x" params="name parent_link *origin">
     <link name="${name}_link">
       <visual>
-        <origin xyz="-0.095 0 0" rpy="${pi/2} 0 -${pi/2}" />
+        <material name="black"/>
         <geometry>
-          <mesh filename="package://clearpath_sensors_description/meshes/novatel_smart7.stl"/>
+          <cylinder radius="0.0305" length="0.0195" />
         </geometry>
-        <material name="novatel_white">
-          <color rgba="0.8 0.8 0.8 1.0" />
-        </material>
       </visual>
       <collision>
-        <origin xyz="-0.095 0 0" rpy="${pi/2} 0 -${pi/2}" />
+        <material name="black"/>
         <geometry>
-          <mesh filename="package://clearpath_sensors_description/meshes/novatel_smart7.stl"/>
+          <cylinder radius="0.0305" length="0.0195" />
         </geometry>
       </collision>

File: clearpath_sensors_description/urdf/novatel_smart6.urdf.xacro (robot description, xacro)
@@ -1,5 +1,5 @@
 <?xml version="1.0"?>
 <robot xmlns:xacro="http://www.ros.org/wiki/xacro">
-  <xacro:macro name="novatel_smart6" params="name">
+  <xacro:macro name="novatel_smart6" params="name parent_link *origin">
     <link name="${name}_link">
       <visual>
@@ -13,4 +13,15 @@
       </visual>
     </link>
+    <joint name="${name}_joint" type="fixed">
+      <child link="${name}_link"/>
+      <parent link="${parent_link}"/>
+      <xacro:insert_block name="origin"/>
+    </joint>
+    <gazebo reference="${name}_link">
+      <sensor name="${name}" type="navsat">
+        <always_on>1</always_on>
+        <update_rate>1</update_rate>
+      </sensor>
+    </gazebo>
   </xacro:macro>
 </robot>
