Commit message: Imported upstream version '0.1.3' of 'upstream'

File: clearpath_mounts_description/urdf/pacs/bracket.urdf.xacro (robot description, xacro)
@@ -79,5 +79,5 @@
           <!-- Add the Bracket-->
           <xacro:bracket_generic name="${name}" parent_link="${parent_link}" mesh="${mesh}" mesh_thickness="${mesh_thickness}" x="${mesh_x}" y="${mesh_y}" z="${mesh_z}">
-              <origin xyz="${bracket_xyz}" rpy="${bracket_rpy}"/>
+              <xacro:insert_block name="origin"/>
           </xacro:bracket_generic>
       </xacro:if>

File: clearpath_platform_description/urdf/a200/a200.urdf.xacro (robot description, xacro)
@@ -161,7 +161,4 @@
         <xacro:unless value="$(arg is_sim)">
           <plugin>clearpath_platform/A200Hardware</plugin>
-          <plugin>fake_components/GenericSystem</plugin>
-          <param name="hw_start_duration_sec">2.0</param>
-          <param name="hw_stop_duration_sec">3.0</param>
           <param name="wheel_diameter">0.3302</param>
           <param name="max_accel">5.0</param>

File: clearpath_platform_description/urdf/j100/j100.urdf.xacro (robot description, xacro)
@@ -183,5 +183,4 @@
         <xacro:unless value="$(arg is_sim)">
           <plugin>clearpath_platform/J100Hardware</plugin>
-          <plugin>fake_components/GenericSystem</plugin>
         </xacro:unless>
       </hardware>
