Commit message: Imported upstream version '0.2.0' of 'upstream'

File: clearpath_mounts_description/urdf/pacs/bracket.urdf.xacro (robot description, xacro)
@@ -26,60 +26,48 @@
       Brackets: add user defined bracket per mount name (i.e. A01)
       - adds extension to increase height of bracket (HUSKY_A01_BRACKET_EXTENSION 0). (e.g. 20, 40, 60, 80)
-      - adds type of bracket (HUSKY_A01_BRACKET_TYPE horizontal). (e.g. horizontal, horizontal_large, vertical)
+      - adds type of bracket (HUSKY_A01_BRACKET_TYPE horizontal). (e.g. horizontal, large, vertical)
       - adds mounting location always as A01_mount
   -->
   <xacro:macro name="bracket" params="name parent_link model:=horizontal *origin">
-      <!-- Check to Add Bracket -->
-      <xacro:property name="name_upper"             value="${name.upper()}"/>
-      <xacro:property name="bracket_enabled"        value="1"/>
-      <xacro:property name="bracket_type"           value="${model}"/>
-      <xacro:property name="bracket_xyz"            value="0 0 0"/>
-      <xacro:property name="bracket_rpy"            value="0 0 0"/>
-      <xacro:property name="bracket_extension"      value="0"/>
-      <xacro:property name="bracket_parent"         value="${name}"/>
-      <xacro:property name="bracket_extension_xyz"  value="${bracket_xyz}"/>
-      <xacro:property name="bracket_extension_rpy"  value="${bracket_rpy}"/>
-      <xacro:if value="${bracket_enabled}">
-          <!-- Horizontal -->
-          <xacro:if value="${bracket_type == 'horizontal'}">
-              <xacro:property name="mesh_x" value="0.09"/>
-              <xacro:property name="mesh_y" value="0.09"/>
-              <xacro:property name="mesh_z" value="0.010125"/>
-              <xacro:property name="mesh_thickness" value="0.010125"/>
-              <xacro:property name="mesh" value="package://clearpath_mounts_description/meshes/pacs/bracket_horizontal.stl"/>
-          </xacro:if>
-          <!-- Horizontal Large -->
-          <xacro:if value="${bracket_type == 'horizontal_large'}">
-              <xacro:property name="mesh_x" value="0.16"/>
-              <xacro:property name="mesh_y" value="0.16"/>
-              <xacro:property name="mesh_z" value="0.00635"/>
-              <xacro:property name="mesh_thickness" value="0.00635"/>
-              <xacro:property name="mesh" value="package://clearpath_mounts_description/meshes/pacs/bracket_horizontal_large.stl"/>
-          </xacro:if>
-          <!-- Vertical -->
-          <xacro:if value="${bracket_type == 'vertical'}">
-              <xacro:property name="mesh_x" value="0.1"/>
-              <xacro:property name="mesh_y" value="0.1"/>
-              <xacro:property name="mesh_z" value="0.1419"/>
-              <xacro:property name="mesh_thickness" value="0.010125"/>
-              <xacro:property name="mesh" value="package://clearpath_mounts_description/meshes/pacs/bracket_vertical.stl"/>
-              <!-- Vertical Mount -->
-              <link name="${name}_vertical_mount"/>
-              <joint name="${name}_vertical_mount_joint" type="fixed">
-                <child link="${name}_vertical_mount"/>
-                <parent link="${name}_mount"/>
-                <origin xyz="0.0518 0 0.086875" rpy="0 -${pi/2} 0"/>
-              </joint>
-          </xacro:if>
-          <xacro:unless value="${bracket_type == 'vertical' or
-                                  bracket_type == 'horizontal' or
-                                  bracket_type == 'horizontal_large'}">
-              ${xacro.error(str("Bracket type (" + str(bracket_enabled) + ") does not exist. Select between 'vertical', 'horizontal', or 'horizontal_large'"))}
-          </xacro:unless>
-          <!-- Add the Bracket-->
-          <xacro:bracket_generic name="${name}" parent_link="${parent_link}" mesh="${mesh}" mesh_thickness="${mesh_thickness}" x="${mesh_x}" y="${mesh_y}" z="${mesh_z}">
-              <xacro:insert_block name="origin"/>
-          </xacro:bracket_generic>
-      </xacro:if>
+    <!-- Horizontal -->
+    <xacro:if value="${model == 'horizontal'}">
+        <xacro:property name="mesh_x" value="0.09"/>
+        <xacro:property name="mesh_y" value="0.09"/>
+        <xacro:property name="mesh_z" value="0.010125"/>
+        <xacro:property name="mesh_thickness" value="0.010125"/>
+        <xacro:property name="mesh" value="package://clearpath_mounts_description/meshes/pacs/bracket_horizontal.stl"/>
+    </xacro:if>
+    <!-- Horizontal Large -->
+    <xacro:if value="${model == 'large'}">
+        <xacro:property name="mesh_x" value="0.16"/>
+        <xacro:property name="mesh_y" value="0.16"/>
+        <xacro:property name="mesh_z" value="0.00635"/>
+        <xacro:property name="mesh_thickness" value="0.00635"/>
+        <xacro:property name="mesh" value="package://clearpath_mounts_description/meshes/pacs/bracket_horizontal_large.stl"/>
+    </xacro:if>
+    <!-- Vertical -->
+    <xacro:if value="${model == 'vertical'}">
+        <xacro:property name="mesh_x" value="0.1"/>
+        <xacro:property name="mesh_y" value="0.1"/>
+        <xacro:property name="mesh_z" value="0.1419"/>
+        <xacro:property name="mesh_thickness" value="0.010125"/>
+        <xacro:property name="mesh" value="package://clearpath_mounts_description/meshes/pacs/bracket_vertical.stl"/>
+        <!-- Vertical Mount -->
+        <link name="${name}_vertical_mount"/>
+        <joint name="${name}_vertical_mount_joint" type="fixed">
+          <child link="${name}_vertical_mount"/>
+          <parent link="${name}_mount"/>
+          <origin xyz="0.0518 0 0.086875" rpy="0 -${pi/2} 0"/>
+        </joint>
+    </xacro:if>
+    <xacro:unless value="${model == 'vertical' or
+                            model == 'horizontal' or
+                            model == 'large'}">
+        ${xacro.error(str("Bracket type (" + str(bracket_enabled) + ") does not exist. Select between 'vertical', 'horizontal', or 'large'"))}
+    </xacro:unless>
+    <!-- Add the Bracket-->
+    <xacro:bracket_generic name="${name}" parent_link="${parent_link}" mesh="${mesh}" mesh_thickness="${mesh_thickness}" x="${mesh_x}" y="${mesh_y}" z="${mesh_z}">
+      <xacro:insert_block name="origin"/>
+    </xacro:bracket_generic>
   </xacro:macro>
   <!--
@@ -89,5 +77,5 @@
     <link name="${name}_link">
       <visual>
-          <material name="dark_grey"/>
+          <material name="clearpath_dark_grey"/>
           <geometry>
             <mesh filename="${mesh}" />

File: clearpath_platform_description/urdf/a200/a200.urdf.xacro (robot description, xacro)
@@ -1,12 +1,12 @@
 <?xml version="1.0"?>
 <robot xmlns:xacro="http://ros.org/wiki/xacro">
-  <xacro:arg name="gazebo_controllers" default="$(find clearpath_control)/config/a200/control.yaml" />
   <xacro:arg name="namespace" default="" />
   <xacro:arg name="is_sim" default="false" />
   <xacro:arg name="serial_port" default="/dev/clearpath/prolific" />
+  <xacro:arg name="gazebo_controllers" default="$(find clearpath_control)/config/a200/control.yaml"/>
   <!-- Included URDF/XACRO Files -->
-  <xacro:include filename="$(find clearpath_platform_description)/urdf/a200/wheel.urdf.xacro" />
+  <xacro:include filename="$(find clearpath_platform_description)/urdf/a200/wheels/wheel.urdf.xacro" />
   <xacro:property name="M_PI" value="3.14159"/>
-  <xacro:macro name="a200">
+  <xacro:macro name="a200" params="wheel:='default'">
     <!-- Base Size -->
     <xacro:property name="base_x_size" value="0.98740000" />
@@ -130,28 +130,14 @@
       <child link="rear_bumper_mount" />
     </joint>
-    <xacro:if value="$(arg is_sim)">
-      <gazebo>
-        <plugin filename="libign_ros2_control-system.so" name="ign_ros2_control::IgnitionROS2ControlPlugin">
-          <parameters>$(arg gazebo_controllers)</parameters>
-          <ros>
-            <remapping>~/odom:=platform/odom</remapping>
-            <remapping>~/cmd_vel_unstamped:=platform/cmd_vel_unstamped</remapping>
-            <remapping>/tf:=tf</remapping>
-            <remapping>/tf_static:=tf_static</remapping>
-            <remapping>/diagnostics:=diagnostics</remapping>
-            <remapping>joint_states:=platform/joint_states</remapping>
-            <namespace>$(arg namespace)</namespace>
-          </ros>
-        </plugin>
-      </gazebo>
-      <gazebo>
-        <plugin filename="libignition-gazebo-pose-publisher-system.so" name="ignition::gazebo::systems::PosePublisher">
-          <publish_link_pose>true</publish_link_pose>
-          <publish_nested_model_pose>true</publish_nested_model_pose>
-          <use_pose_vector_msg>true</use_pose_vector_msg>
-          <update_frequency>50</update_frequency>
-        </plugin>
-      </gazebo>
-    </xacro:if>
+    <!-- Default mount -->
+    <link name="default_mount"/>
+    <joint name="default_mount_joint" type="fixed">
+      <child link="default_mount"/>
+      <parent link="base_link"/>
+      <origin xyz="0.0 0.0 0.224"/>
+    </joint>
+    <!-- Gazebo Controller -->
+    <xacro:include filename="$(find clearpath_platform_description)/urdf/generic/gazebo.urdf.xacro"/>
+    <!-- ROS2 controls -->
     <ros2_control name="a200_hardware" type="system">
       <hardware>

File: clearpath_platform_description/urdf/a200/attachments/bumper.urdf.xacro (robot description, xacro)
@@ -1,9 +1,5 @@
 <?xml version="1.0"?>
 <robot xmlns:xacro="http://ros.org/wiki/xacro">
-    <xacro:macro name="bumper" params="name extension:=0 *origin">
-        <xacro:property name="parent_link" value="front_bumper_mount" />
-        <xacro:if value="${'rear' in name}" >
-            <xacro:property name="parent_link" value="rear_bumper_mount" />
-        </xacro:if>
+    <xacro:macro name="bumper" params="name model:='default' parent_link:='front_bumper_mount' extension:=0 *origin">
         <!-- Spawn bumper link -->
         <link name="${name}_link">
@@ -15,8 +11,14 @@
         </link>
         <xacro:unless value="${extension > 0}">
+            <link name="${name}_base_link"/>
+            <joint name="${name}_base_joint" type="fixed">
+                <xacro:insert_block name="origin"/>
+                <parent link="${parent_link}"/>
+                <child link="${name}_base_link"/>
+            </joint>
             <!-- Attach bumper -->
             <joint name="${name}_joint" type="fixed">
                 <origin xyz="0.075 0 0" rpy="0 0 0" />
-                <parent link="${parent_link}" />
+                <parent link="${name}_base_link" />
                 <child link="${name}_link" />
             </joint>
@@ -28,5 +30,5 @@
                         <cylinder radius="0.0095" length="${extension}" />
                     </geometry>
-                    <material name="dark_grey" />
+                    <material name="clearpath_dark_grey" />
                     <origin xyz="${extension / 2} 0 0" rpy="0 ${M_PI/2} 0" />
                 </visual>
@@ -37,22 +39,28 @@
                         <cylinder radius="0.0095" length="${extension}" />
                     </geometry>
-                    <material name="dark_grey" />
+                    <material name="clearpath_dark_grey" />
                     <origin xyz="${extension / 2} 0 0" rpy="0 ${M_PI/2} 0" />
                 </visual>
             </link>
+            <link name="${name}_base_link"/>
             <link name="${name}_extension_mount"/>
+            <joint name="${name}_base_joint" type="fixed">
+                <xacro:insert_block name="origin"/>
+                <parent link="${parent_link}"/>
+                <child link="${name}_base_link"/>
+            </joint>
             <joint name="${name}_extension_joint_1" type="fixed">
                 <origin xyz="0 0.1084 0" rpy="0 0 0" />
-                <parent link="${parent_link}" />
+                <parent link="${name}_base_link" />
                 <child link="${name}_extension_link_1" />
             </joint>
             <joint name="${name}_extension_joint_2" type="fixed">
                 <origin xyz="0 -0.1084 0" rpy="0 0 0" />
-                <parent link="${parent_link}" />
+                <parent link="${name}_base_link" />
                 <child link="${name}_extension_link_2" />
             </joint>
             <joint name="${name}_extension_mount_joint" type="fixed">
                 <origin xyz="${extension} 0 0" rpy="0 0 0" />
-                <parent link="${parent_link}" />
+                <parent link="${name}_base_link" />
                 <child link="${name}_extension_mount" />
             </joint>

File: clearpath_platform_description/urdf/a200/attachments/top_plate.urdf.xacro (robot description, xacro)
@@ -1,11 +1,11 @@
 <?xml version="1.0"?>
 <robot xmlns:xacro="http://ros.org/wiki/xacro">
-    <!-- <xacro:include filename="$(find clearpath_platform_description)/urdf/common.urdf.xacro" /> -->
-    <xacro:macro name="top_plate" params="model:=default *origin">
-        <!-- Spawn the top plate -->
+    <xacro:macro name="top_plate" params="name model:=default parent_link:=default_mount *origin">
+      <!-- Large Model -->
       <xacro:if value="${model == 'large'}">
-        <link name="top_plate_link">
+        <!-- Spawn top plate -->
+        <link name="${name}_link">
           <visual>
-            <origin xyz="0 0 0" rpy="0 0 0" />
+            <origin xyz="0.0812 0 0" rpy="0 0 0" />
             <geometry>
               <mesh filename="package://clearpath_platform_description/meshes/a200/attachments/large_top_plate.dae" />
@@ -13,5 +13,5 @@
           </visual>
           <collision>
-            <origin xyz="0 0 0" rpy="0 0 0"/>
+            <origin xyz="0.0812 0 0" rpy="0 0 0"/>
             <geometry>
               <mesh filename="package://clearpath_platform_description/meshes/a200/attachments/large_top_plate_collision.stl" />
@@ -20,28 +20,45 @@
         </link>
         <!-- Attach top plate -->
-        <joint name="top_plate_joint" type="fixed">
-          <parent link="base_link" />
-          <child link="top_plate_link"/>
-          <origin xyz="0.0812 0 0.225" rpy="0 0 0"/>
+        <joint name="${name}_joint" type="fixed">
+          <parent link="${parent_link}" />
+          <child link="${name}_link"/>
+          <xacro:insert_block name="origin"/>
         </joint>
         <!-- Top plate front link -->
-        <joint name="top_plate_front_joint" type="fixed">
-          <parent link="top_plate_link" />
-          <child link="top_plate_front_link"/>
+        <link name="${name}_front_mount"/>
+        <joint name="${name}_front_joint" type="fixed">
+          <parent link="${name}_link" />
+          <child link="${name}_front_mount"/>
           <origin xyz="0.4125 0 0.00672" rpy="0 0 0"/>
         </joint>
         <!-- Top plate rear link-->
-        <joint name="top_plate_rear_joint" type="fixed">
-          <parent link="top_plate_link" />
-          <child link="top_plate_rear_link"/>
+        <link name="${name}_rear_mount"/>
+        <joint name="${name}_rear_joint" type="fixed">
+          <parent link="${name}_link" />
+          <child link="${name}_rear_mount"/>
           <origin xyz="-0.4125 0 0.00672" rpy="0 0 0"/>
         </joint>
-        <link name="top_plate_front_link"/>
-        <link name="top_plate_rear_link"/>
       </xacro:if>
+      <!-- Default Model -->
       <xacro:if value="${model == 'default'}">
-        <link name="top_plate_link">
+        <!-- Spawn user rails -->
+        <link name="${name}_user_rail_link">
           <visual>
-            <origin xyz="0 0 0" rpy="0 0 0" />
+            <origin xyz="0.272 0 0.019"/>
+            <geometry>
+              <mesh filename="package://clearpath_platform_description/meshes/a200/attachments/user_rail.dae" />
+            </geometry>
+          </visual>
+        </link>
+        <!-- Attach user rails to base link -->
+        <joint name="${name}_user_rail_joint" type="fixed">
+          <xacro:insert_block name="origin"/>
+          <parent link="${parent_link}" />
+          <child link="${name}_user_rail_link" />
+        </joint>
+        <!-- Spawn top plate -->
+        <link name="${name}_link">
+          <visual>
+            <origin xyz="0.0812 0 0" rpy="0 0 0" />
             <geometry>
               <mesh filename="package://clearpath_platform_description/meshes/a200/attachments/top_plate.dae" />
@@ -49,5 +66,5 @@
           </visual>
           <collision>
-            <origin xyz="0 0 0" rpy="0 0 0"/>
+            <origin xyz="0.0812 0 0" rpy="0 0 0"/>
             <geometry>
               <mesh filename="package://clearpath_platform_description/meshes/a200/attachments/top_plate.stl" />
@@ -56,42 +73,31 @@
         </link>
         <!-- Attach top plate -->
-        <joint name="top_plate_joint" type="fixed">
-          <parent link="base_link" />
-          <child link="top_plate_link"/>
-          <origin xyz="0.0812 0 0.245" rpy="0 0 0"/>
+        <joint name="${name}_joint" type="fixed">
+          <parent link="${name}_user_rail_link" />
+          <child link="${name}_link"/>
+          <origin xyz="0 0 0.021" rpy="0 0 0"/>
         </joint>
         <!-- Top plate front link -->
-        <joint name="top_plate_front_joint" type="fixed">
-          <parent link="top_plate_link" />
-          <child link="top_plate_front_link"/>
+        <link name="${name}_front_mount"/>
+        <joint name="${name}_front_joint" type="fixed">
+          <parent link="${name}_link" />
+          <child link="${name}_front_mount"/>
           <origin xyz="0.36367 0 0.00639" rpy="0 0 0"/>
         </joint>
         <!-- Top plate rear link-->
-        <joint name="top_plate_rear_joint" type="fixed">
-          <parent link="top_plate_link" />
-          <child link="top_plate_rear_link"/>
+        <link name="${name}_rear_mount"/>
+        <joint name="${name}_rear_joint" type="fixed">
+          <parent link="${name}_link" />
+          <child link="${name}_rear_mount"/>
           <origin xyz="-0.36633 0 0.00639" rpy="0 0 0"/>
         </joint>
-        <!-- Spawn user rails -->
-        <link name="user_rail_link">
+      </xacro:if>
+      <!-- PACS Model -->
+      <xacro:if value="${model == 'pacs'}">
+        <!-- Spawn top plate -->
+        <link name="${name}_link">
           <visual>
-            <geometry>
-              <mesh filename="package://clearpath_platform_description/meshes/a200/attachments/user_rail.dae" />
-            </geometry>
-          </visual>
-        </link>
-        <!-- Attach user rails to base link -->
-        <joint name="user_rail" type="fixed">
-          <origin xyz="0.272 0 0.245" rpy="0 0 0" />
-          <parent link="base_link" />
-          <child link="user_rail_link" />
-        </joint>
-        <link name="top_plate_front_link"/>
-        <link name="top_plate_rear_link"/>
-      </xacro:if>
-      <xacro:if value="${model == 'pacs'}">
-        <link name="top_plate_link">
-          <visual>
-            <material name="dark_grey" />
+            <origin xyz="0.0483 0 0"/>
+            <material name="clearpath_dark_grey" />
             <geometry>
               <mesh filename="package://clearpath_platform_description/meshes/a200/attachments/pacs_top_plate.stl" />
@@ -99,21 +105,21 @@
           </visual>
           <collision>
-            <material name="dark_grey" />
-            <origin xyz="0 0 0.00317500531673" rpy="0 0 0"/>
+            <material name="clearpath_dark_grey" />
+            <origin xyz="0.0483 0 0.003175" rpy="0 0 0"/>
             <geometry>
-              <box size="0.670000076294 0.590000033379 0.00635001063347"/>
+              <box size="0.67 0.59 0.00635"/>
             </geometry>
           </collision>
         </link>
         <!-- Attach PACS top plate -->
-        <joint name="top_plate_joint" type="fixed">
-          <child link="top_plate_link"/>
-          <parent link="base_link"/>
-          <origin xyz="0.048299998045 0 0.227500006557" rpy="0 0 0"/>
+        <joint name="${name}_joint" type="fixed">
+          <child link="${name}_link"/>
+          <parent link="${parent_link}"/>
+          <xacro:insert_block name="origin"/>
         </joint>
         <!-- Generate PACS mounts -->
         <xacro:full_mounts
-          name="top_plate"
-          parent_link="top_plate_link"
+          name="${name}"
+          parent_link="${name}_link"
           column="a"
           row="1"
@@ -124,6 +130,6 @@
           z="0.00635" />
         <xacro:full_mounts
-          name="top_plate"
-          parent_link="top_plate_link"
+          name="${name}"
+          parent_link="${name}_link"
           column="a"
           row="3"
@@ -134,6 +140,6 @@
           z="0.00635" />
         <xacro:full_mounts
-          name="top_plate"
-          parent_link="top_plate_link"
+          name="${name}"
+          parent_link="${name}_link"
           column="g"
           row="3"
@@ -144,6 +150,6 @@
           z="0.00635" />
         <xacro:full_mounts
-          name="top_plate"
-          parent_link="top_plate_link"
+          name="${name}"
+          parent_link="${name}_link"
           column="a"
           row="7"

File: clearpath_platform_description/urdf/j100/attachments/top_plate.urdf.xacro (robot description, xacro)
@@ -1,7 +1,7 @@
 <?xml version="1.0"?>
 <robot xmlns:xacro="http://ros.org/wiki/xacro">
-    <xacro:macro name="top_plate" params="model:=default">
+    <xacro:macro name="top_plate" params="name:=ark_enclosure model:=default parent_link:=default_mount *origin">
       <xacro:if value="${model == 'ark_enclosure'}">
-         <link name="ark_enclosure_link">
+         <link name="${name}_link">
           <visual>
             <origin xyz="0 0 0" rpy="0 0 0"/>
@@ -9,10 +9,11 @@
               <mesh filename="package://clearpath_platform_description/meshes/j100/attachments/ark_enclosure.stl"/>
             </geometry>
-            <material name="dark_grey" />
+            <material name="clearpath_dark_grey" />
           </visual>
         </link>
-        <joint name="ark_enclosure_joint" type="fixed">
-          <parent link="mid_mount" />
-          <child link="ark_enclosure_link" />
+        <joint name="${name}_joint" type="fixed">
+          <parent link="${parent_link}" />
+          <child link="${name}_link" />
+          <xacro:insert_block name="origin"/>
         </joint>
       </xacro:if>
