Commit message: Rebase from 'release/humble/clearpath_platform_description'

File: urdf/a200/attachments/sensor_arch.urdf.xacro (robot description, xacro)
@@ -1,8 +1,8 @@
 <?xml version="1.0"?>
-<robot xmlns:xacro="http://ros.org/wiki/xacro" name="510_mm_sensor_arch">
-  <xacro:macro name="structure" params="parent_link model:=sensor_arch_510 *origin">
+<robot xmlns:xacro="http://ros.org/wiki/xacro" name="sensor_arch">
+  <xacro:macro name="sensor_arch" params="name parent_link:=default_mount model:=sensor_arch_510 *origin">
     <xacro:if value="${model == 'sensor_arch_510'}">
       <!-- Spawn the sensor arch link -->
-      <link name="sensor_arch_link">
+      <link name="${name}_link">
         <visual>
           <origin xyz="0 0 0.51" rpy="0 0 0"/>
@@ -18,20 +18,20 @@
         </collision>
       </link>
-      <link name="sensor_arch_mount"/>
+      <link name="${name}_mount"/>
       <!-- Attach the sensor arch to the top plate -->
-      <joint name="sensor_arch_joint" type="fixed">
+      <joint name="${name}_joint" type="fixed">
         <xacro:insert_block name="origin"/>
         <parent link="${parent_link}"/>
-        <child link="sensor_arch_link"/>
+        <child link="${name}_link"/>
       </joint>
       <joint name="sensor_arch_mount_joint" type="fixed">
         <origin xyz="0 0 0.51" rpy="0 0 0"/>
-        <parent link="sensor_arch_link"/>
-        <child link="sensor_arch_mount"/>
+        <parent link="${name}_link"/>
+        <child link="${name}_mount"/>
       </joint>
     </xacro:if>
     <xacro:if value="${model == 'sensor_arch_300'}">
       <!-- Spawn the sensor arch link -->
-      <link name="sensor_arch_link">
+      <link name="${name}_link">
         <visual>
           <origin xyz="0 0 0.3" rpy="0 0 0"/>
@@ -47,15 +47,15 @@
         </collision>
       </link>
-      <link name="sensor_arch_mount"/>
+      <link name="${name}_mount"/>
       <!-- Attach the sensor arch to the top plate -->
-      <joint name="sensor_arch_joint" type="fixed">
+      <joint name="${name}_joint" type="fixed">
         <xacro:insert_block name="origin"/>
         <parent link="${parent_link}"/>
-        <child link="sensor_arch_link"/>
+        <child link="${name}_link"/>
       </joint>
-      <joint name="sensor_arch_mount_joint" type="fixed">
+      <joint name="${name}_mount_joint" type="fixed">
         <origin xyz="0 0 0.3" rpy="0 0 0"/>
-        <parent link="sensor_arch_link"/>
-        <child link="sensor_arch_mount"/>
+        <parent link="${name}_link"/>
+        <child link="${name}_mount"/>
       </joint>
     </xacro:if>

File: urdf/j100/attachments/fender.urdf.xacro (robot description, xacro)
@@ -1,7 +1,7 @@
 <?xml version="1.0"?>
 <robot xmlns:xacro="http://ros.org/wiki/xacro">
-  <xacro:macro name="rear_fender" params="model *origin">
+  <xacro:macro name="fender" params="name model parent_link:=base_link *origin">
     <!-- Spawn fender link -->
-    <link name="rear_fender_link">
+    <link name="${name}_link">
       <visual>
         <geometry>
@@ -13,20 +13,20 @@
           </xacro:if>
         </geometry>
-        <material name="yellow" />
+        <material name="clearpath_yellow" />
       </visual>
     </link>
     <xacro:if value="${model == 'sensor'}">
-      <link name="rear_fender_mount"/>
-      <joint name="rear_fender_mount_joint" type="fixed">
+      <link name="${name}_mount"/>
+      <joint name="${name}_mount_joint" type="fixed">
         <origin xyz="0.25629 0 0.07455" rpy="${pi} 0 0" />
-        <parent link="rear_fender_link" />
-        <child link="rear_fender_mount" />
+        <parent link="${name}_link" />
+        <child link="${name}_mount" />
       </joint>
     </xacro:if>
     <!-- Attach fender -->
-    <joint name="rear_fender_joint" type="fixed">
-      <origin xyz="0 0 0" rpy="0 0 ${pi}"/>
-      <parent link="base_link" />
-      <child link="rear_fender_link" />
+    <joint name="${name}_joint" type="fixed">
+      <xacro:insert_block name="origin"/>
+      <parent link="${parent_link}" />
+      <child link="${name}_link" />
     </joint>
   </xacro:macro>

File: urdf/j100/wheels/wheel.urdf.xacro (robot description, xacro)
@@ -1,4 +1,4 @@
 <?xml version="1.0"?>
-<robot xmlns:xacro="http://ros.org/wiki/xacro" name="a200_wheel">
+<robot xmlns:xacro="http://ros.org/wiki/xacro" name="j100_wheel">
   <xacro:macro name="j100_wheel" params="prefix *joint_pose">
     <link name="${prefix}_wheel_link">
@@ -8,5 +8,5 @@
           <mesh filename="package://clearpath_platform_description/meshes/j100/j100_wheel.stl"/>
         </geometry>
-        <material name="black" />
+        <material name="clearpath_black" />
       </visual>
       <collision>
@@ -35,15 +35,4 @@
       <axis xyz="0 1 0" />
     </joint>
-    <!-- In reality, J100 has only two motors, one per side. However, it's more
-         straightforward for Gazebo to simulate as if there's an actuator per wheel. -->
-    <transmission name="${prefix}_wheel_trans">
-      <type>transmission_interface/SimpleTransmission</type>
-      <joint name="${prefix}_wheel">
-        <hardwareInterface>hardware_interface/VelocityJointInterface</hardwareInterface>
-      </joint>
-      <actuator name="${prefix}_actuator">
-        <mechanicalReduction>1</mechanicalReduction>
-      </actuator>
-    </transmission>
   </xacro:macro>
 </robot>
