Commit message: Rebase from 'upstream'

File: clearpath_platform_description/urdf/links/mesh.urdf.xacro (robot description, xacro)
@@ -5,5 +5,5 @@
       <visual>
         <geometry>
-          <mesh filename="file://${visual}"/>
+          <mesh filename="${visual}"/>
         </geometry>
         <material name="clearpath_dark_grey"/>
