Commit message: Imported upstream version '2.1.0' of 'upstream'

File: clearpath_manipulators_description/urdf/arm/universal_robots.urdf.xacro (robot description, xacro)
@@ -2,5 +2,5 @@
 <robot xmlns:xacro="http://ros.org/wiki/xacro">
   <xacro:arg name="is_sim" default="false"/>
-  <xacro:arg name="use_fake_hardware" default="false"/>
+  <xacro:arg name="use_mock_hardware" default="false"/>
   <xacro:arg name="use_manipulation_controllers" default="false"/>
   <xacro:include filename="$(find ur_description)/urdf/ur_macro.xacro"/>
@@ -19,5 +19,4 @@
     safety_pos_margin:=''
     safety_k_position:=''
-    generate_ros2_control_tag:=''
     headless_mode:=''
     robot_ip:=''
@@ -42,6 +41,6 @@
     tool_device_name:=''
     tool_tcp_port:=''
-    use_fake_hardware:=''
-    fake_sensor_commands:=''
+    use_mock_hardware:=''
+    mock_sensor_commands:=''
     sim_gazebo:=''
     sim_ignition:=''
@@ -58,5 +57,4 @@
     <xacro:property name="_safety_k_position" value="20" lazy_eval="false"/>
     <!-- Default ros2_control Parameters -->
-    <xacro:property name="_generate_ros2_control_tag" value="$(arg use_manipulation_controllers)" lazy_eval="false"/>
     <xacro:property name="_headless_mode" value="false" lazy_eval="false"/>
     <xacro:property name="_robot_ip" value="192.168.131.40" lazy_eval="false"/>
@@ -83,6 +81,6 @@
     <xacro:property name="_tool_tcp_port" value="54321" lazy_eval="false"/>
     <!-- Default Simulation Parameters -->
-    <xacro:property name="_use_fake_hardware" value="false" />
-    <xacro:property name="_fake_sensor_commands" value="false" />
+    <xacro:property name="_use_mock_hardware" value="false" />
+    <xacro:property name="_mock_sensor_commands" value="false" />
     <xacro:property name="_sim_gazebo" value="false" />
     <xacro:property name="_sim_ignition" value="$(arg is_sim)" />
@@ -98,5 +96,4 @@
     <xacro:if value="${safety_pos_margin != ''}"> <xacro:property name="_safety_pos_margin" value="${safety_pos_margin}" lazy_eval="false"/> </xacro:if>
     <xacro:if value="${safety_k_position != ''}"> <xacro:property name="_safety_k_position" value="${safety_k_position}" lazy_eval="false"/> </xacro:if>
-    <xacro:if value="${generate_ros2_control_tag != ''}"> <xacro:property name="_generate_ros2_control_tag" value="${generate_ros2_control_tag}" lazy_eval="false"/> </xacro:if>
     <xacro:if value="${headless_mode != ''}"> <xacro:property name="_headless_mode" value="${headless_mode}" lazy_eval="false"/> </xacro:if>
     <xacro:if value="${robot_ip != ''}"> <xacro:property name="_robot_ip" value="${robot_ip}" lazy_eval="false"/> </xacro:if>
@@ -121,14 +118,12 @@
     <xacro:if value="${tool_device_name != ''}"> <xacro:property name="_tool_device_name" value="${tool_device_name}" lazy_eval="false"/> </xacro:if>
     <xacro:if value="${tool_tcp_port != ''}"> <xacro:property name="_tool_tcp_port" value="${tool_tcp_port}" lazy_eval="false"/> </xacro:if>
-    <xacro:if value="${use_fake_hardware != ''}"> <xacro:property name="_use_fake_hardware" value="${use_fake_hardware}" lazy_eval="false"/> </xacro:if>
-    <xacro:if value="${fake_sensor_commands != ''}"> <xacro:property name="_fake_sensor_commands" value="${fake_sensor_commands}" lazy_eval="false"/> </xacro:if>
+    <xacro:if value="${use_mock_hardware != ''}"> <xacro:property name="_use_mock_hardware" value="${use_mock_hardware}" lazy_eval="false"/> </xacro:if>
+    <xacro:if value="${mock_sensor_commands != ''}"> <xacro:property name="_mock_sensor_commands" value="${mock_sensor_commands}" lazy_eval="false"/> </xacro:if>
     <xacro:if value="${sim_gazebo != ''}"> <xacro:property name="_sim_gazebo" value="${sim_gazebo}" lazy_eval="false"/> </xacro:if>
     <xacro:if value="${sim_ignition != ''}"> <xacro:property name="_sim_ignition" value="${sim_ignition}" lazy_eval="false"/> </xacro:if>
-    <!-- Universal_Robots_ROS2_Description -->
     <xacro:ur_robot
       name="${name}"
+      tf_prefix="${_tf_prefix}"
       parent="${parent_link}"
-      tf_prefix="${_tf_prefix}"
-      initial_positions="${_initial_positions}"
       joint_limits_parameters_file="${_joint_limits_parameters_file}"
       kinematics_parameters_file="${_kinematics_parameters_file}"
@@ -138,33 +133,39 @@
       safety_pos_margin="${_safety_pos_margin}"
       safety_k_position="${_safety_k_position}"
-      generate_ros2_control_tag="${_generate_ros2_control_tag}"
-      headless_mode="${_headless_mode}"
-      robot_ip="${_robot_ip}"
-      script_filename="${_script_filename}"
-      output_recipe_filename="${_output_recipe_filename}"
-      input_recipe_filename="${_input_recipe_filename}"
-      reverse_ip="${_reverse_ip}"
-      script_command_port="${_script_command_port}"
-      reverse_port="${_reverse_port}"
-      script_sender_port="${_script_sender_port}"
-      trajectory_port="${_trajectory_port}"
-      transmission_hw_interface="${_transmission_hw_interface}"
-      non_blocking_read="{_non_blocking_read}"
-      use_tool_communication="${_use_tool_communication}"
-      tool_voltage="${_tool_voltage}"
-      tool_parity="${_tool_parity}"
-      tool_baud_rate="${_tool_baud_rate}"
-      tool_stop_bits="${_tool_stop_bits}"
-      tool_rx_idle_chars="${_tool_rx_idle_chars}"
-      tool_tx_idle_chars="${_tool_tx_idle_chars}"
-      tool_device_name="${_tool_device_name}"
-      tool_tcp_port="${_tool_tcp_port}"
-      use_fake_hardware="${_use_fake_hardware}"
-      fake_sensor_commands="${_fake_sensor_commands}"
-      sim_gazebo="${_sim_gazebo}"
-      sim_ignition="${_sim_ignition}"
       >
       <xacro:insert_block name="origin"/>
     </xacro:ur_robot>
+    <!-- Universal_Robots_ROS2_Driver HardwareInterface -->
+    <xacro:if value="$(arg use_manipulation_controllers)">
+      <xacro:include filename="$(find ur_robot_driver)/urdf/ur.ros2_control.xacro" />
+      <xacro:ur_ros2_control
+        name="${name}"
+        tf_prefix="${_tf_prefix}"
+        kinematics_parameters_file="${_kinematics_parameters_file}"
+        transmission_hw_interface="${_transmission_hw_interface}"
+        use_mock_hardware="${_use_mock_hardware}"
+        mock_sensor_commands="${_mock_sensor_commands}"
+        headless_mode="${_headless_mode}"
+        initial_positions="${_initial_positions}"
+        use_tool_communication="${_use_tool_communication}"
+        tool_voltage="${_tool_voltage}"
+        tool_parity="${_tool_parity}"
+        tool_baud_rate="${_tool_baud_rate}"
+        tool_stop_bits="${_tool_stop_bits}"
+        tool_rx_idle_chars="${_tool_rx_idle_chars}"
+        tool_tx_idle_chars="${_tool_tx_idle_chars}"
+        tool_device_name="${_tool_device_name}"
+        tool_tcp_port="${_tool_tcp_port}"
+        robot_ip="${_robot_ip}"
+        script_filename="${_script_filename}"
+        output_recipe_filename="${_output_recipe_filename}"
+        input_recipe_filename="${_input_recipe_filename}"
+        reverse_ip="${_reverse_ip}"
+        script_command_port="${_script_command_port}"
+        reverse_port="${_reverse_port}"
+        script_sender_port="${_script_sender_port}"
+        trajectory_port="${_trajectory_port}"
+      />
+    </xacro:if>
   </xacro:macro>
 </robot>
